Commit message: 장애물을 돌아가는 경로 계획: RRT-Connect 직접 구현 + MoveIt2 비교
문서에 '경로 계획은 없다' 고 적어 둔 구멍을 메웠다.

- sim/plan_rrt.py: 관절 공간 RRT-Connect + 무작위 단축 + 재샘플. 충돌 판정은 트윈 실행기가 쓰는 것을 그대로 부른다
  (계획기와 실행기가 다른 기준을 보면 '계획은 됐는데 돌리면 부딪힌다'). 가짜 팔 2D 문제로 pytest 6건
- tools/twin_path_plan.py: 같은 이동 48건(2층 + 목적지 6개 적재, 4시드)에서 직선 vs 계획 비교 —
  직선 34/48(71%) → 계획 48/48(100%), 계획 중앙 85 ms, 돌아가는 값 +0.25 s, 재검사 전건 무충돌
- ros2_ws/src/robotsim_moveit_config: MoveIt2 계획 전용 move_group 설정(SRDF·kinematics·limits·OMPL) +
  plan_compare 노드. 같은 URDF·같은 장면·같은 시작·목표로 48/48 성공, 계획 11 ms, 경로 평균 10.24 vs 10.61 rad
- twin_closed_loop --plan / twin_server --plan: 직선이 막히면 계획으로 돌아간다. 폐루프 60박스 결과는 불변(75%) —
  실행기가 이미 IK 해를 바꿔 피하고 있었다는 뜻이고, 그대로 기록했다
- URDF 에 충돌 형상 추가(MoveIt 이 자기·장면 충돌을 보려면 필요), docs/30 §14 · docs/42 6-f · 실험로그 71·72
- pytest 104

File: ros2_ws/src/twin_bridge/urdf/ur10e_track.urdf (robot description, URDF)
Before this commit: robot ur10e_track, 13 links, 12 joints
Links:
- link carriage: geometry collision cylinder length=0.0600 radius=0.1800; visual cylinder length=0.0600 radius=0.1800
- link forearm_link: geometry collision cylinder length=0.5710 radius=0.0750; visual cylinder length=0.5710 radius=0.0750
- link pedestal: geometry collision cylinder length=1.0800 radius=0.1600; visual cylinder length=1.0800 radius=0.1600
- link rail: geometry collision cylinder length=0.0600 radius=0.0500; visual cylinder length=0.0600 radius=0.0500
- link shoulder_link: geometry collision cylinder length=0.1760 radius=0.0750; visual cylinder length=0.1760 radius=0.0750
- link tool: geometry collision cylinder length=0.1500 radius=0.0500; visual cylinder length=0.1500 radius=0.0500
- link upper_arm_link: geometry collision cylinder length=0.6281 radius=0.0750; visual cylinder length=0.6281 radius=0.0750
- link ur_base: geometry collision cylinder length=0.1200 radius=0.0800; visual cylinder length=0.1200 radius=0.0800
- link wrist_1_link: geometry collision cylinder length=0.1350 radius=0.0500; visual cylinder length=0.1350 radius=0.0500
- link wrist_2_link: geometry collision cylinder length=0.1200 radius=0.0500; visual cylinder length=0.1200 radius=0.0500
- link wrist_3_link: geometry collision cylinder length=0.1000 radius=0.0500; visual cylinder length=0.1000 radius=0.0500
